Commit message: Modified launch files

File: description/lidar.xacro (robot description, xacro)
@@ -2,5 +2,5 @@
 <robot xmlns:xacro="http://www.ros.org/wiki/xacro">
     <joint name="lidar_joint" type='fixed'>
-        <parent link="chassis"/>
+        <parent link="chassis_link"/>
         <child link="lidar_link"/>
         <origin xyz="0 0 0.205" rpy="0 0 0"/>
@@ -11,5 +11,5 @@
                 <cylinder radius="0.1" length="0.05"/>
             </geometry>
-            <origin xyz="0 0 0" rpy="1.57 0 0"/>
+            <origin xyz="0 0 0" rpy="0 0 0"/>
             <material name="black"/>
         </visual>
@@ -18,5 +18,5 @@
                 <cylinder radius="0.1" length="0.05"/>
             </geometry>
-            <origin xyz="0 0 0" rpy="1.57 0 0"/>
+            <origin xyz="0 0 0" rpy="0 0 0"/>
         </collision>
          <xacro:inertial_cylinder mass="0.05" length="0.05" radius="1.0">
@@ -24,3 +24,31 @@
         </xacro:inertial_cylinder>
     </link>
+    <gazebo reference="lidar_link">
+        <material>Gazebo/black</material>
+        <sensor name="laser" type="ray">
+            <pose> 0 0 0 0 0 0 </pose>
+            <visualize>true</visualize>
+            <update_rate>10</update_rate>
+            <ray>
+                <scan>
+                    <horizontal>
+                        <samples>360</samples>
+                        <min_angle>-3.14</min_angle>
+                        <max_angle>3.14</max_angle>
+                    </horizontal>
+                </scan>
+                <range>
+                    <min>0.3</min>
+                    <max>12</max>
+                </range>
+            </ray>
+            <plugin name="laser_controller" filename="libgazebo_ros_ray_sensor.so">
+                <ros>
+                    <argument>~/out:=scan</argument>
+                </ros>
+                <output_type>sensor_msgs/LaserScan</output_type>
+                <frame_name>laser_frame</frame_name>
+            </plugin>
+        </sensor>
+    </gazebo>
 </robot>

File: description/robot.urdf.xacro (robot description, xacro)
@@ -1,6 +1,12 @@
 <?xml version="1.0"?>
 <robot xmlns:xacro="http://www.ros.org/wiki/xacro"  name="robot">
+    <xacro:arg name="use_ros2_control" default="true"/>
     <xacro:include filename="robot_core.xacro" />
-    <xacro:include filename="control.xacro"/>
-    <xacro:include filename="lidar.xacro"/>
+    <xacro:if value="$(arg use_ros2_control)">
+        <xacro:include filename="ros2_control.xacro" />
+    </xacro:if>
+    <xacro:unless value="$(arg use_ros2_control)">
+        <xacro:include filename="gazebo_control.xacro" />
+    </xacro:unless>
+    <xacro:include filename="lidar.xacro" />
 </robot>

File: description/robot_core.xacro (robot description, xacro)
@@ -17,7 +17,4 @@
         <color rgba="0.7 0 0 1"/>
     </material>
-    <material name="silver">
-        <color rgba="0.75 0.75 0.75"/>
-    </material>
     <link name="base_link">
     </link>
@@ -28,5 +25,5 @@
             </geometry>
             <origin xyz = "0 0 0.1" rpy="0 0 0" />
-            <material name="silver"/>
+            <material name="grey"/>
         </visual>
         <collision>
@@ -46,9 +43,9 @@
             </geometry>
             <origin xyz="0 0 0" rpy="1.57 0 0"/>
-            <material name="black"/>
+            <material name="grey"/>
         </visual>
         <collision>
             <geometry>
-                <cylinder radius="0.1" length="0.05"/>
+                <sphere radius="0.1"/>
             </geometry>
             <origin xyz="0 0 0" rpy="1.57 0 0"/>
@@ -64,9 +61,9 @@
             </geometry>
             <origin xyz="0 0 0" rpy="1.57 0 0"/>
-            <material name="black"/>
+            <material name="grey"/>
         </visual>
         <collision>
             <geometry>
-                <cylinder radius="0.1" length="0.05"/>
+                <sphere radius="0.1"/>
             </geometry>
             <origin xyz="0 0 0" rpy="1.57 0 0"/>
@@ -82,5 +79,5 @@
             </geometry>
             <origin xyz="0 0 0" rpy="0 0 0" />
-            <material name="silver"/>
+            <material name="red"/>
         </visual>
         <collision>
@@ -100,5 +97,5 @@
             </geometry>
             <origin xyz="0 0 0" rpy="0 0 0" />
-            <material name="silver"/>
+            <material name="green"/>
         </visual>
         <collision>
